Commit message: added pos and vel limits in sahr.urdf

File: resources/robots/sahr/urdf/sahr.urdf (robot description, URDF)
Before this commit: robot SAHR_v76, 93 links, 92 joints
Joints:
- joint head_pitch: limit effort=6 velocity=0 -> effort=6 velocity=50
- joint head_yaw: limit effort=6 velocity=0 -> effort=6 velocity=50
- joint left_ankle_pitch: limit effort=6 velocity=0 -> lower=-0.8 upper=1.0 effort=6 velocity=50
- joint left_ankle_roll: limit effort=6 velocity=0 -> lower=-0.5 upper=0.5 effort=6 velocity=50
- joint left_elbow: limit effort=6 velocity=0 -> effort=6 velocity=50
- joint left_hip_pitch: limit lower=0 upper=0 effort=6 velocity=0 -> lower=-2.1 upper=1.0 effort=6 velocity=50
- joint left_hip_roll: limit effort=6 velocity=0 -> lower=-0.6 upper=0.6 effort=6 velocity=50
- joint left_hip_yaw: limit effort=6 velocity=0 -> lower=-0.5 upper=1.5 effort=6 velocity=50
- joint left_knee: limit lower=0 upper=1.5 effort=6 velocity=0 -> lower=0 upper=1.5 effort=6 velocity=50
- joint left_shoulder_pitch: limit effort=6 velocity=0 -> effort=6 velocity=50
- joint left_shoulder_roll: limit effort=6 velocity=0 -> effort=6 velocity=50
- joint right_ankle_pitch: limit effort=6 velocity=0 -> lower=-0.8 upper=1.0 effort=6 velocity=50
- joint right_ankle_roll: limit effort=6 velocity=0 -> lower=-0.5 upper=0.5 effort=6 velocity=50
- joint right_elbow: limit effort=6 velocity=0 -> effort=6 velocity=50
- joint right_hip_pitch: limit lower=0 upper=0 effort=6 velocity=0 -> lower=-2.1 upper=1.0 effort=6 velocity=50
- joint right_hip_roll: limit effort=6 velocity=0 -> lower=-0.6 upper=0.6 effort=6 velocity=50
- joint right_hip_yaw: limit effort=6 velocity=0 -> lower=-0.5 upper=1.5 effort=6 velocity=50
- joint right_knee: limit lower=0 upper=1.5 effort=6 velocity=0 -> lower=0 upper=1.5 effort=6 velocity=50
- joint right_shoulder_pitch: limit effort=6 velocity=0 -> effort=6 velocity=50
- joint right_shoulder_roll: limit effort=6 velocity=0 -> effort=6 velocity=50
